File: CAD-files/bme280Breakout.kicad_pcb (KiCad board)
At the start: 2 copper layers, 12.7 x 12.7 mm, 9 parts, among them J1 Conn_01x04_Male, U1 BME280

Commit message: added castellated holes
Parts:
- J1: value Conn_01x04_Male -> Castellated_Conn_01x04; footprint Connector_PinHeader_2.54mm:PinHeader_1x04_P2.54mm_Vertical -> DS-connectors:Castellated_PinHeader_01x04_P2.54mm_Vertical
- moved J1 2.57 mm to (141.0, 108.3)
- turned C1 to 180 degrees
- turned C2 to 180 degrees
Connections:
- J1 pad 1: +3V3 -> GND
- J1 pad 2: GND -> +3V3
Routing:
- net GND: track 16.8 -> 20.5 mm
Other:
- board text added: "3V3"
- board text removed: "+3V3"

Commit message: Add files via upload
Parts:
- added J2: Castellated_Conn_01x01, DS-connectors:Castellated_PinHeader_01x01_P2.54mm_Vertical, F.Cu at (141.5, 98.7)
- added J3: Castellated_Conn_01x01, DS-connectors:Castellated_PinHeader_01x01_P2.54mm_Vertical, F.Cu at (149.1, 98.7)
- C1, C2: footprint Capacitor_SMD:C_0603_1608Metric -> Capacitor_SMD:C_0805_2012Metric
- R1, R2, R3, R4: footprint Resistor_SMD:R_0603_1608Metric -> Resistor_SMD:R_0805_2012Metric
- moved C1 0.51 mm to (143.8, 103.6)
- moved R1 0.51 mm to (150.9, 104.5)
- moved R4 0.38 mm to (147.3, 104.0)
- moved R2 0.25 mm to (150.9, 102.5)
Routing:
- net GND: track 20.5 -> 30.0 mm
- net +3V3: track 29.2 -> 31.0 mm
- net SDO: track 5.15 -> 5.85 mm

Commit message: Add files via upload
Parts:
- added kibuzzard-62094851: G***, kibuzzard-62094851, F.Cu at (144.9, 97.9)
- added kibuzzard-62094851: G***, kibuzzard-62094851, B.Cu at (149.7, 98.0)
- added kibuzzard-6209486A: G***, kibuzzard-6209486A, F.Cu at (145.9, 97.9)
- added kibuzzard-6209486A: G***, kibuzzard-6209486A, B.Cu at (148.7, 98.0)
- added kibuzzard-62094872: G***, kibuzzard-62094872, F.Cu at (146.9, 97.9)
- added kibuzzard-62094872: G***, kibuzzard-62094872, B.Cu at (147.7, 98.0)
- added kibuzzard-62094878: G***, kibuzzard-62094878, F.Cu at (147.8, 97.9)
- added kibuzzard-62094878: G***, kibuzzard-62094878, B.Cu at (146.8, 98.0)
- added kibuzzard-62094881: G***, kibuzzard-62094881, F.Cu at (148.7, 97.9)
- added kibuzzard-62094881: G***, kibuzzard-62094881, B.Cu at (145.9, 98.0)
- added kibuzzard-62094889: G***, kibuzzard-62094889, F.Cu at (149.7, 97.9)
- added kibuzzard-62094889: G***, kibuzzard-62094889, B.Cu at (145.0, 98.0)
- added kibuzzard-62094948: G***, kibuzzard-62094948, F.Cu at (147.3, 98.9)
- added kibuzzard-620949A9: G***, kibuzzard-620949A9, F.Cu at (143.5, 107.1)
- added kibuzzard-620949BC: G***, kibuzzard-620949BC, F.Cu at (143.5, 106.3)
- added kibuzzard-620949C8: G***, kibuzzard-620949C8, F.Cu at (143.5, 105.5)
- added kibuzzard-620949C8: G***, kibuzzard-620949C8, F.Cu at (148.6, 106.3)
- added kibuzzard-620949D5: G***, kibuzzard-620949D5, F.Cu at (146.1, 105.5)
- added kibuzzard-620949D5: G***, kibuzzard-620949D5, F.Cu at (146.1, 107.1)
- added kibuzzard-620949E0: G***, kibuzzard-620949E0, F.Cu at (146.1, 106.3)
- added kibuzzard-620949FF: G***, kibuzzard-620949FF, F.Cu at (151.1, 107.1)
- added kibuzzard-620949FF: G***, kibuzzard-620949FF, F.Cu at (148.6, 107.1)
- added kibuzzard-62094A0D: G***, kibuzzard-62094A0D, F.Cu at (148.6, 105.5)
- added kibuzzard-62094A25: G***, kibuzzard-62094A25, F.Cu at (151.1, 106.3)
- added kibuzzard-62094A2C: G***, kibuzzard-62094A2C, F.Cu at (151.1, 105.5)
- added kibuzzard-62094C34: G***, kibuzzard-62094C34, B.Cu at (145.7, 99.1)
- added kibuzzard-62094C8E: G***, kibuzzard-62094C8E, B.Cu at (147.3, 99.9)
- added kibuzzard-62094D35: G***, kibuzzard-62094D35, B.Cu at (147.3, 101.0)
- added kibuzzard-62094D47: G***, kibuzzard-62094D47, B.Cu at (147.3, 101.9)
- added kibuzzard-62094DBA: G***, kibuzzard-62094DBA, B.Cu at (147.3, 106.3)
- added kibuzzard-62094DDC: G***, kibuzzard-62094DDC, B.Cu at (141.7, 103.5)
- added kibuzzard-62094E12: G***, kibuzzard-62094E12, B.Cu at (148.9, 99.1)
- added kibuzzard-62094E24: G***, kibuzzard-62094E24, B.Cu at (144.2, 99.5)
- added kibuzzard-62094E24: G***, kibuzzard-62094E24, B.Cu at (147.3, 99.4)
- added kibuzzard-62095084: G***, kibuzzard-62095084, B.Cu at (147.3, 103.3)
Routing:
- net +3V3: track 31.0 -> 31.9 mm
Other:
- net class Default removed
- board text removed: "3.3V Only!"
- board text removed: "3V3"
- board text removed: "@DeepSpace00"
- board text removed: "BME280"
- board text removed: "Default I2C Addr 0x77"
- board text removed: "Destination SPACE Inc."
- board text removed: "GND"
- board text removed: "Pres/Hum/Temp"
- board text removed: "SCL"
- board text removed: "SDA"
- board text removed: "Temp, Pressure Humidity"
